Commit message: improve grasping (still has some flaws)

File: src/agilus_robotiq_description/urdf/agilus_robotiq.urdf.xacro (robot description, xacro)
@@ -68,8 +68,17 @@
     <xacro:arm_joint num="5" init="0.0"/>
     <xacro:arm_joint num="6" init="0.0"/>
-    <!-- gripper: single actuated knuckle + 5 mimic joints. gz_ros2_control
-         applies the mimic coupling in software (the default physics engine does
-         NOT enforce URDF mimic constraints), so the followers must be declared
-         here with mimic params. Only the knuckle gets a command interface. -->
+    <!-- gripper: single actuated knuckle + 5 mimic joints, driven by a
+         POSITION command. gz_ros2_control implements position commands as
+         velocity setpoints (joint_velocity = position_proportional_gain *
+         error * update_rate), so the fingers are kinematically driven; the
+         followers are coupled by the gz_ros2_control SOFTWARE mimic (URDF
+         <mimic> tags; gz-sim's URDF->SDF conversion drops <mimic>, so physics
+         mimic is not available, and effort control of a software-mimicked
+         chain locks the knuckle — hence position control). When the fingers
+         block on an object, the controller goal never completes; the grasp
+         skill detects the stall and cancels the goal so the controller holds
+         the fingers at the object's width. The object is held by the
+         geometric trap (fingers locked narrower than the object) plus contact
+         friction — a physical grip, no virtual attachment. -->
     <joint name="${prefix}robotiq_85_left_knuckle_joint">
       <command_interface name="position">
@@ -122,22 +131,8 @@
     </plugin>
   </gazebo>
-  <!-- ============ grasp: detachable-joint attach on close ============ -->
-  <!-- bullet-featherstone ignores <ode> friction, so reliable pick uses a
-       DetachableJoint: starts detached, attaches red_cube to the left
-       fingertip on /gripper/attach, releases on /gripper/detach.
-       NOTE: gz-sim8 ignores <suppress_initial_attach> — its attachRequested
-       flag defaults to true, so the plugin welds red_cube to the fingertip
-       on the first physics tick after spawn. The spawn launch file undoes
-       this (detach + pose reset) a few seconds after the robot spawns. -->
-  <gazebo>
-    <plugin filename="gz-sim-detachable-joint-system"
-            name="gz::sim::systems::DetachableJoint">
-      <parent_link>robotiq_85_left_finger_tip_link</parent_link>
-      <child_model>red_cube</child_model>
-      <child_link>link</child_link>
-      <attach_topic>/gripper/attach</attach_topic>
-      <detach_topic>/gripper/detach</detach_topic>
-      <output_topic>/gripper/attach_state</output_topic>
-    </plugin>
-  </gazebo>
+  <!-- ============ grasp: physical grip, no virtual attachment ============ -->
+  <!-- The gripper is position-servo driven (see the comment on the knuckle
+       joint above); on an object the grasp skill holds the fingers at the
+       object's width (geometric trap + friction). The DetachableJoint that
+       used to weld red_cube to the fingertip is gone. -->
 </robot>

Commit message: improve grasping

File: src/agilus_robotiq_description/urdf/agilus_robotiq.urdf.xacro (robot description, xacro)
@@ -77,8 +77,7 @@
          chain locks the knuckle — hence position control). When the fingers
          block on an object, the controller goal never completes; the grasp
-         skill detects the stall and cancels the goal so the controller holds
-         the fingers at the object's width. The object is held by the
-         geometric trap (fingers locked narrower than the object) plus contact
-         friction — a physical grip, no virtual attachment. -->
+         skill detects the stall and leaves a small over-close command active
+         so the controller maintains normal force. The object is held by
+         physical contact friction — no virtual attachment. -->
     <joint name="${prefix}robotiq_85_left_knuckle_joint">
       <command_interface name="position">

File: src/agilus_robotiq_description/urdf/robotiq_2f_85_macro_collisionfix.urdf.xacro (robot description, xacro)
@@ -132,7 +132,13 @@
             </visual>
             <collision>
-                <origin xyz="0.0 0.0 0.0165" rpy="0 0 0" />
-                <geometry>
-                    <box size="0.012 0.018 0.033" />
+                <!-- Bounding box of left_finger_tip.dae.  This mesh is
+                     asymmetric: its inner face reaches 25.26 mm toward the
+                     object, while the former centred 12 mm collision box
+                     reached only 6 mm.  That discrepancy is why the visual
+                     claw could be deeply inside a cube after physics had
+                     already detected contact. -->
+                <origin xyz="-0.0096407 -0.0008000 0.0225077" rpy="0 0 0" />
+                <geometry>
+                    <box size="0.0312358 0.0270000 0.0570155" />
                 </geometry>
                 <surface>
@@ -168,7 +174,8 @@
             </visual>
             <collision>
-                <origin xyz="0.0 0.0 0.0165" rpy="0 0 0" />
-                <geometry>
-                    <box size="0.012 0.018 0.033" />
+                <!-- Mirrored bounding box of right_finger_tip.dae. -->
+                <origin xyz="0.0096407 0.0000500 0.0225077" rpy="0 0 0" />
+                <geometry>
+                    <box size="0.0312358 0.0270000 0.0570155" />
                 </geometry>
                 <surface>

Commit message: added grasp fix gz plugin to not have to focus on physical gripping issues anymore

File: src/agilus_robotiq_description/urdf/agilus_robotiq.urdf.xacro (robot description, xacro)
@@ -129,9 +129,30 @@
       <parameters>$(arg controller_config)</parameters>
     </plugin>
+    <!-- Gazebo Harmonic port of gazebo_grasp_fix: when both fingertip contact
+         sensors touch the same dynamic object, the plugin creates a fixed
+         detachable joint to the gripper base. It removes that joint once both
+         contacts have been absent long enough for the gripper to open. -->
+    <plugin filename="libnlra_gz_grasp_fix.so" name="nlra::systems::GraspFix">
+      <!-- The fixed base joint is reduced into link_6 during URDF->SDF conversion. -->
+      <palm_link>${prefix}link_6</palm_link>
+      <left_finger_link>${prefix}robotiq_85_left_finger_tip_link</left_finger_link>
+      <right_finger_link>${prefix}robotiq_85_right_finger_tip_link</right_finger_link>
+      <left_contact_sensor>left_grasp_contact</left_contact_sensor>
+      <right_contact_sensor>right_grasp_contact</right_contact_sensor>
+      <grip_count_threshold>10</grip_count_threshold>
+      <release_count_threshold>20</release_count_threshold>
+    </plugin>
   </gazebo>
-  <!-- ============ grasp: physical grip, no virtual attachment ============ -->
-  <!-- The gripper is position-servo driven (see the comment on the knuckle
-       joint above); on an object the grasp skill holds the fingers at the
-       object's width (geometric trap + friction). The DetachableJoint that
-       used to weld red_cube to the fingertip is gone. -->
+  <!-- Contact data for the grasp-fix system. The names match the explicit
+       fingertip collision names in the Robotiq macro. -->
+  <gazebo reference="${prefix}robotiq_85_left_finger_tip_link">
+    <sensor name="left_grasp_contact" type="contact">
+      <contact><collision>${prefix}robotiq_85_left_finger_tip_link_collision</collision></contact>
+    </sensor>
+  </gazebo>
+  <gazebo reference="${prefix}robotiq_85_right_finger_tip_link">
+    <sensor name="right_grasp_contact" type="contact">
+      <contact><collision>${prefix}robotiq_85_right_finger_tip_link_collision</collision></contact>
+    </sensor>
+  </gazebo>
 </robot>

File: src/agilus_robotiq_description/urdf/robotiq_2f_85_macro_collisionfix.urdf.xacro (robot description, xacro)
@@ -30,5 +30,5 @@
                 </geometry>
             </visual>
-            <collision>
+            <collision name="${prefix}robotiq_85_left_finger_tip_link_collision">
                 <geometry>
                     <box size="0.048 0.048 0.052" />
@@ -71,5 +71,5 @@
                 </geometry>
             </visual>
-            <collision>
+            <collision name="${prefix}robotiq_85_right_finger_tip_link_collision">
                 <origin xyz="0.0 0.0 0.022" rpy="0 0 0" />
                 <geometry>

Commit message: moveit: full NL pick-and-place completes 10/10 on fresh boot
- gripper: physics-only mimic (restore <mimic> tags + mimic="false"
  attributes on ros2_control follower joints) — deterministic follower
  tracking; dual-mimic conflict (physics + software) removed
- fix_start_state: true for jazzy CheckStartStateBounds (joint_4 limit
  overshoot at lower:blue_box)
- TOOL0_FINGERTIP_OFFSET=0.098: world-model grasp poses are fingertip-
  midpoint heights; planner drives tool0 (98 mm above fingertips) — was
  descending below the tabletop, grasp missed the cube
- verified: 'put the cube into the box' -> success=True, cube at target
  (xy dist 0.7 cm) on fresh boot

File: src/agilus_robotiq_description/urdf/agilus_robotiq.urdf.xacro (robot description, xacro)
@@ -91,5 +91,5 @@
       <state_interface name="effort"/>
     </joint>
-    <joint name="${prefix}robotiq_85_right_knuckle_joint">
+    <joint name="${prefix}robotiq_85_right_knuckle_joint" mimic="false">
       <param name="mimic">${prefix}robotiq_85_left_knuckle_joint</param>
       <param name="multiplier">-1</param>
@@ -97,5 +97,5 @@
       <state_interface name="velocity"/>
     </joint>
-    <joint name="${prefix}robotiq_85_left_inner_knuckle_joint">
+    <joint name="${prefix}robotiq_85_left_inner_knuckle_joint" mimic="false">
       <param name="mimic">${prefix}robotiq_85_left_knuckle_joint</param>
       <param name="multiplier">1</param>
@@ -103,5 +103,5 @@
       <state_interface name="velocity"/>
     </joint>
-    <joint name="${prefix}robotiq_85_right_inner_knuckle_joint">
+    <joint name="${prefix}robotiq_85_right_inner_knuckle_joint" mimic="false">
       <param name="mimic">${prefix}robotiq_85_left_knuckle_joint</param>
       <param name="multiplier">-1</param>
@@ -109,5 +109,5 @@
       <state_interface name="velocity"/>
     </joint>
-    <joint name="${prefix}robotiq_85_left_finger_tip_joint">
+    <joint name="${prefix}robotiq_85_left_finger_tip_joint" mimic="false">
       <param name="mimic">${prefix}robotiq_85_left_knuckle_joint</param>
       <param name="multiplier">-1</param>
@@ -115,5 +115,5 @@
       <state_interface name="velocity"/>
     </joint>
-    <joint name="${prefix}robotiq_85_right_finger_tip_joint">
+    <joint name="${prefix}robotiq_85_right_finger_tip_joint" mimic="false">
       <param name="mimic">${prefix}robotiq_85_left_knuckle_joint</param>
       <param name="multiplier">1</param>
